File: PCBs/191126RvW-WateringSystemPICAXE/191126RvW-WateringSystemPICAXE.sch (KiCad schematic (older format))
At the start: 17 parts, among them J1 MotorConn, J2 SerIn, J3 SerSelect, J4 SerOut, J5 Screw_Terminal_01x04, J6 SerSelect, Q1 KN2222A, U1 PICAXEM2

Commit message: New board size
Parts:
- U1: symbol PICAXE:PICAXEM2 -> 191126RvW-WateringSystemPICAXE-rescue:PICAXEM2-PICAXE
Changed lines of the file:
@@
 Connection ~ 2450 1550
 $Comp
-L PICAXE:PICAXEM2 U1
+L 191126RvW-WateringSystemPICAXE-rescue:PICAXEM2-PICAXE U1
 U 1 1 5DE64F40
 P 6300 1200

Commit message: pcb changes
Connections:
- net GNDPWR is gone; now on net GNDD: J1.1 (Pin_1), J5.2 (Pin_2), Q1.1 (E)
Changed lines of the file:
@@
 $EndComp
 Wire Wire Line
-	8800 1050 8800 1200
+	8800 1050 8800 1100
 Wire Wire Line
-	9150 1050 9150 1200
+	9150 1050 9150 1100
 Wire Wire Line
 	9500 1050 9500 1300
@@
 Wire Wire Line
 	5350 1750 5300 1750
+Wire Wire Line
+	8800 1100 9150 1100
+Connection ~ 8800 1100
+Wire Wire Line
+	8800 1100 8800 1200
+Connection ~ 9150 1100
+Wire Wire Line
+	9150 1100 9150 1200
 $EndSCHEMATC
