File: PCBs/EightRelayModule/EightRelayModule.sch (KiCad schematic (older format))
At the start: 18 parts, among them J2 Programmer, J3 PowerForHardReset, J4 Power, J5 RelayModule, Q101 2N7000, Q102 2N7000, Q103 2N7000, U1 PICAXEM2, U2 MAX485

Commit message: Made PCB
Parts:
- C1: footprint (none) -> Capacitor_THT:C_Disc_D4.3mm_W1.9mm_P5.00mm
- C2: footprint (none) -> Capacitor_THT:CP_Radial_D13.0mm_P5.00mm
- D1: footprint (none) -> Diode_THT:D_T-1_P10.16mm_Horizontal
- J2: footprint (none) -> Connector_PinHeader_2.54mm:PinHeader_1x04_P2.54mm_Vertical
- J3: footprint (none) -> Connector_PinHeader_2.54mm:PinHeader_1x02_P2.54mm_Vertical
- J4: footprint (none) -> Connector_Wago:Wago_734-133_1x03_P3.50mm_Vertical
- J5: footprint (none) -> Connector_PinHeader_2.54mm:PinHeader_1x10_P2.54mm_Vertical
- R1, R101, R102, R103, R2, R3: footprint (none) -> Resistor_THT:R_Axial_DIN0411_L9.9mm_D3.6mm_P15.24mm_Horizontal
- U1: footprint (none) -> Package_DIP:DIP-8_W7.62mm; symbol PICAXEs:PICAXEM2 -> PICAXE:PICAXEM2
- U2: symbol RvWsymbols:MAX485 -> RvWSymbols:MAX485
Changed lines of the file:
@@
 EESchema Schematic File Version 4
+LIBS:PICAXE
+LIBS:RvWSymbols
+LIBS:EightRelayModule-cache
 EELAYER 30 0
 EELAYER END
@@
 $EndDescr
 $Comp
-L PICAXEs:PICAXEM2 U1
+L PICAXE:PICAXEM2 U1
 U 1 1 6232FC9E
 P 4350 1850
 F 0 "U1" H 4600 1850 50  0000 C CNN
 F 1 "PICAXEM2" H 4575 1750 50  0000 C CNN
-F 2 "" H 4350 1850 50  0001 C CNN
+F 2 "Package_DIP:DIP-8_W7.62mm" H 4350 1850 50  0001 C CNN
 F 3 "" H 4350 1850 50  0001 C CNN
 	1    4350 1850
@@
 F 0 "D1" V 2954 2930 50  0000 L CNN
 F 1 "D" V 3045 2930 50  0000 L CNN
-F 2 "" H 3000 2850 50  0001 C CNN
+F 2 "Diode_THT:D_T-1_P10.16mm_Horizontal" H 3000 2850 50  0001 C CNN
 F 3 "~" H 3000 2850 50  0001 C CNN
 	1    3000 2850
@@
 F 0 "R1" H 3068 3296 50  0000 L CNN
 F 1 "1k" H 3068 3205 50  0000 L CNN
-F 2 "" V 3040 3240 50  0001 C CNN
+F 2 "Resistor_THT:R_Axial_DIN0411_L9.9mm_D3.6mm_P15.24mm_Horizontal" V 3040 3240 50  0001 C CNN
 F 3 "~" H 3000 3250 50  0001 C CNN
 	1    3000 3250
@@
 F 0 "R2" V 2645 2225 50  0000 C CNN
 F 1 "22k" V 2736 2225 50  0000 C CNN
-F 2 "" V 2890 2215 50  0001 C CNN
+F 2 "Resistor_THT:R_Axial_DIN0411_L9.9mm_D3.6mm_P15.24mm_Horizontal" V 2890 2215 50  0001 C CNN
 F 3 "~" H 2850 2225 50  0001 C CNN
 	1    2850 2225
@@
 F 0 "R3" H 2543 2421 50  0000 L CNN
 F 1 "10k" H 2543 2330 50  0000 L CNN
-F 2 "" V 2515 2365 50  0001 C CNN
+F 2 "Resistor_THT:R_Axial_DIN0411_L9.9mm_D3.6mm_P15.24mm_Horizontal" V 2515 2365 50  0001 C CNN
 F 3 "~" H 2475 2375 50  0001 C CNN
 	1    2475 2375
@@
 F 0 "J2" H 1908 1631 50  0000 C CNN
 F 1 "Programmer" H 1908 1540 50  0000 C CNN
-F 2 "" H 1800 1350 50  0001 C CNN
+F 2 "Connector_PinHeader_2.54mm:PinHeader_1x04_P2.54mm_Vertical" H 1800 1350 50  0001 C CNN
 F 3 "~" H 1800 1350 50  0001 C CNN
 	1    1800 1350
@@
 F 0 "J3" H 4008 1581 50  0000 C CNN
 F 1 "PowerForHardReset" H 4008 1490 50  0000 C CNN
-F 2 "" H 3900 1400 50  0001 C CNN
+F 2 "Connector_PinHeader_2.54mm:PinHeader_1x02_P2.54mm_Vertical" H 3900 1400 50  0001 C CNN
 F 3 "~" H 3900 1400 50  0001 C CNN
 	1    3900 1400
@@
 F 0 "C1" H 4985 1604 50  0000 R CNN
 F 1 "100nF" H 4985 1695 50  0000 R CNN
-F 2 "" H 5138 1500 50  0001 C CNN
+F 2 "Capacitor_THT:C_Disc_D4.3mm_W1.9mm_P5.00mm" H 5138 1500 50  0001 C CNN
 F 3 "~" H 5100 1650 50  0001 C CNN
 	1    5100 1650
@@
 F 0 "C2" H 7193 1296 50  0000 L CNN
 F 1 "100uF" H 7193 1205 50  0000 L CNN
-F 2 "" H 7113 1100 50  0001 C CNN
+F 2 "Capacitor_THT:CP_Radial_D13.0mm_P5.00mm" H 7113 1100 50  0001 C CNN
 F 3 "~" H 7075 1250 50  0001 C CNN
 	1    7075 1250
@@
 Wire Wire Line
 	9350 3625 9350 3775
-$Comp
-L RvWsymbols:MAX485 U2
-U 1 1 623A65DA
-P 4000 3275
-F 0 "U2" H 3787 3215 50  0000 C CNN
-F 1 "MAX485" H 3787 3124 50  0000 C CNN
-F 2 "RvWfootprints:MAX485" H 4000 3275 50  0001 C CNN
-F 3 "" H 4000 3275 50  0001 C CNN
-	1    4000 3275
-	1    0    0    -1
-$EndComp
 Wire Wire Line
 	3375 3775 3375 3675
-Connection ~ 3375 3675
 Wire Wire Line
 	3375 3575 3000 3575
@@
 F 0 "R101" H 6568 3196 50  0000 L CNN
 F 1 "1k2" H 6568 3105 50  0000 L CNN
-F 2 "" V 6540 3140 50  0001 C CNN
+F 2 "Resistor_THT:R_Axial_DIN0411_L9.9mm_D3.6mm_P15.24mm_Horizontal" V 6540 3140 50  0001 C CNN
 F 3 "~" H 6500 3150 50  0001 C CNN
 	1    6500 3150
@@
 F 0 "R102" H 7468 3221 50  0000 L CNN
 F 1 "1k2" H 7468 3130 50  0000 L CNN
-F 2 "" V 7440 3165 50  0001 C CNN
+F 2 "Resistor_THT:R_Axial_DIN0411_L9.9mm_D3.6mm_P15.24mm_Horizontal" V 7440 3165 50  0001 C CNN
 F 3 "~" H 7400 3175 50  0001 C CNN
 	1    7400 3175
@@
 F 0 "R103" H 8318 3221 50  0000 L CNN
 F 1 "1k2" H 8318 3130 50  0000 L CNN
-F 2 "" V 8290 3165 50  0001 C CNN
+F 2 "Resistor_THT:R_Axial_DIN0411_L9.9mm_D3.6mm_P15.24mm_Horizontal" V 8290 3165 50  0001 C CNN
 F 3 "~" H 8250 3175 50  0001 C CNN
 	1    8250 3175
@@
 F 0 "J5" H 9797 4007 50  0000 R CNN
 F 1 "RelayModule" H 9797 4098 50  0000 R CNN
-F 2 "" H 9825 4125 50  0001 C CNN
+F 2 "Connector_PinHeader_2.54mm:PinHeader_1x10_P2.54mm_Vertical" H 9825 4125 50  0001 C CNN
 F 3 "~" H 9825 4125 50  0001 C CNN
 	1    9825 4125
@@
 F 0 "J4" H 8255 1667 50  0000 L CNN
 F 1 "Power" H 8255 1576 50  0000 L CNN
-F 2 "" H 8175 1625 50  0001 C CNN
+F 2 "Connector_Wago:Wago_734-133_1x03_P3.50mm_Vertical" H 8175 1625 50  0001 C CNN
 F 3 "~" H 8175 1625 50  0001 C CNN
 	1    8175 1625
@@
 Wire Wire Line
 	7500 1525 7975 1525
+$Comp
+L RvWSymbols:MAX485 U2
+U 1 1 623A65DA
+P 4000 3275
+F 0 "U2" H 3787 3215 50  0000 C CNN
+F 1 "MAX485" H 3787 3124 50  0000 C CNN
+F 2 "RvWfootprints:MAX485" H 4000 3275 50  0001 C CNN
+F 3 "" H 4000 3275 50  0001 C CNN
+	1    4000 3275
+	1    0    0    -1
+$EndComp
 $EndSCHEMATC
